Commit message: my
robo

File: myrobotws/src/my_pr_robot/urdf/pr_robot_links_and_joints.urdf (robot description, URDF)
Before this commit: robot pr_robot, 4 links, 3 joints
Joints:
- joint joint1_base_link_to_link1: limit lower=0 upper=4 effort=1000.0 velocity=0.5 -> lower=0 upper=4.0 effort=1000 velocity=0.5
- joint joint2_link1_to_link2: limit lower=-3.14 upper=3.14 effort=1000.0 velocity=1 -> lower=-3.14 upper=3.14 effort=1000 velocity=1.0
- joint joint3_link2_to_hand: axis (none) -> 0 0 0; limit (none) -> lower=0 upper=0 effort=0 velocity=0

File: myrobotws/src/my_pr_robot/urdf/pr_robot_links_and_joints.xacro (robot description, xacro)
@@ -1,84 +1,36 @@
 <?xml version="1.0" ?>
 <robot name = "pr_robot" xmlns:xacro="http://www.ros.org/wiki/xacro">
-    <link name = "base_link">
-    <visual>
-        <origin rpy = "0 0 0" xyz = "0 0 2.5" />
-        <geometry>
-            <cylinder radius = "1.5" length  = "5" />
-        </geometry>
-    </visual>
-    <collision>
-      <origin rpy="0 0 0" xyz="0 0 2.5" />
-      <geometry>
-        <cylinder radius = "1.5" length  = "5" />
-      </geometry>
-    </collision>
-    </link>
-    <joint name = "joint1_base_link_to_link1" type = "prismatic">
-        <parent link = "base_link"/>
-        <child link = "link1"/>
-        <axis xyz = "0 0 1"/>
-        <origin rpy = "0 0 0" xyz = "0 0 1" />
-        <limit effort = "1000.0" lower = "0" upper = "4" velocity="0.5"/>
-    </joint>
-    <link name = "link1">
-    <visual>
-        <origin rpy = "0 0 0" xyz = "0 0 2.5" />
-        <geometry>
-          <cylinder radius = "1" length  = "5" />
-        </geometry>
-	<material name="green">
-    	  <color rgba="0.0 1.0 0.0 1.0"/>
-        </material>
-    </visual>
-    <collision>
-      <origin rpy = "0 0 0" xyz = "0 0 2.5" />
-      <geometry>
-        <cylinder radius = "1" length  = "5" />
-      </geometry>
-    </collision>
-    </link>
-    <joint name = "joint2_link1_to_link2" type = "revolute">
-        <parent link = "link1"/>
-        <child link = "link2"/>
-        <axis xyz = "0 0 1"/>
-        <origin rpy = "0 0 0" xyz = "0 0 0" />
-        <limit effort = "1000.0" lower = "-3.14" upper = "3.14" velocity="1"/>
-    </joint>
-    <link name = "link2">
-    <visual>
-        <origin rpy = "0 0 0" xyz = "2.5 0 5.5" />
-        <geometry>
-            <box size = "5 1 1"/>
-        </geometry>
-    </visual>
-    <collision>
-      <origin rpy = "0 0 0" xyz = "2.5 0 5.5" />
-      <geometry>
-        <box size = "5 1 1"/>
-      </geometry>
-    </collision>
-    </link>
-    <joint name="joint3_link2_to_hand" type="fixed">
-      <origin rpy="0 0 0" xyz="0 0 0"/>
-      <parent link="link2"/>
-      <child link="hand"/>
-    </joint>
-    <link name="hand">
-    <visual>
-      <origin rpy="0 0 0" xyz="5.5 0 5.5" />
-      <geometry>
-        <box size="1 1 1" />
-      </geometry>
-      <material name="green">
-    	<color rgba="0.0 1.0 0.0 1.0"/>
-      </material>
-    </visual>
-    <collision>
-      <origin rpy="0 0 0" xyz="5.5 0 5.5" />
-      <geometry>
-        <box size="1 1 1" />
-      </geometry>
-    </collision>
-</link>
-  </robot>
+  <!-- BGN - Include -->
+  <xacro:include filename="$(find my_pr_robot)/urdf/links_joints.xacro"/>
+  <!-- END - Include -->
+    <my_cylinder_link_red name = "base_link"
+                      origin_rpy = "0 0 0" origin_xyz = "0 0 2.5"
+                      radius = "1.5" length = "5"/>
+    <my_joint name = "joint1_base_link_to_link1"
+              type = "prismatic"
+              origin_rpy = "0 0 0" origin_xyz = "0 0 1"
+              parent = "base_link" child = "link1"
+              axis_xyz = "0 0 1"
+              limit_e = "1000" limit_l = "0" limit_u = "4.0" limit_v = "0.5"/>
+    <my_cylinder_link_green name = "link1"
+                      origin_rpy = "0 0 0" origin_xyz = "0 0 2.5"
+                      radius = "1" length = "5"/>
+    <my_joint name = "joint2_link1_to_link2"
+              type = "revolute"
+              origin_rpy = "0 0 0" origin_xyz = "0 0 0"
+              parent = "link1" child = "link2"
+              axis_xyz = "0 0 1"
+              limit_e = "1000" limit_l = "-3.14" limit_u = "3.14" limit_v = "1.0"/>
+    <my_box_link_red name = "link2"
+                 origin_rpy = "0 0 0" origin_xyz = "2.5 0 5.5"
+                 size = "5 1 1"/>
+    <my_joint name = "joint3_link2_to_hand"
+              type = "fixed"
+              origin_rpy = "0 0 0" origin_xyz = "0 0 0"
+              parent = "link2" child = "hand"
+              axis_xyz = "0 0 0"
+              limit_e = "0" limit_l = "0" limit_u = "0" limit_v = "0"/>
+    <my_box_link_green name = "hand"
+                 origin_rpy = "0 0 0" origin_xyz = "5.5 0 5.5"
+                 size = "1 1 1"/>
+</robot>
